File: line_sensor/line_sensor.kicad_pcb (KiCad board)
At the start: 2 copper layers, 95 x 27 mm, 63 parts, among them J1 Conn_01x06_Socket, Q101 DMG1012T, U1 ITR8307, U101 ITR8307, U102 ITR8307, U103 ITR8307, U104 ITR8307, U105 ITR8307, U106 ITR8307, U107 ITR8307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

Commit message: Feat: some improvments
Parts:
- moved D1 21.0 mm to (152.3, 99.7), turned to 90 degrees
- moved R103 17.4 mm to (154.4, 99.7), turned to 90 degrees
- moved C4 16.7 mm to (153.4, 102.4), turned to 180 degrees
- moved Q101 6.54 mm to (164.3, 104.8), turned to 90 degrees
- moved R101 0.35 mm to (164.5, 107.9), turned to 90 degrees
Routing:
- net +3V3: track 254.6 -> 266.7 mm
- net Earth: track 37.8 -> 40.2 mm

Commit message: Feat: fabrication files using JLCPCB plugin
Parts:
- moved G*** 0.45 mm to (179.8, 100.7)
