File: seebum_esp32s3/seebum_esp32s3.kicad_pcb (KiCad board)
At the start: 4 copper layers, 65 x 56 mm, 90 parts, among them J101 Conn_01x02_Pin, J102 Conn_01x04_Pin, J103 Conn_01x02_Pin, J201 USB_C_Receptacle_USB2.0_16P, J202 USB_C_Receptacle_USB2.0_16P, J203 Conn_02x10_Odd_Even, J204 Conn_02x10_Odd_Even, J401 GPIO, Q101 AO4407, Q201 UMH3N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

Commit message: Feat: fix uart1 schematic issue and I2C redundancy
Parts:
- removed the G*** at (132.4, 76.6)
- removed the G*** at (170.3, 94.6)
- removed R102, R103: 4k7, Resistor_SMD:R_0805_2012Metric
- added G***: LOGO, LOGO, B.Cu at (132.4, 76.5)
- added G***: LOGO, LOGO, B.Cu at (170.6, 94.6)
- added JP101: SolderJumper_2_Open, Jumper:SolderJumper-2_P1.3mm_Open_TrianglePad1.0x1.5mm, F.Cu at (169.5, 87.0)
- added JP102: SolderJumper_2_Open, Jumper:SolderJumper-2_P1.3mm_Open_TrianglePad1.0x1.5mm, F.Cu at (167.0, 87.0)
- J401: moved to B.Cu
- moved R212 9.31 mm to (162.9, 87.0)
- moved R211 5.43 mm to (164.8, 87.0)
- moved J401 2.54 mm to (126.5, 63.3), turned to -90 degrees
- moved JP206 1.50 mm to (139.2, 100.0)
- moved JP207 1.50 mm to (136.7, 100.0)
- moved G*** 0.40 mm to (151.1, 93.7)
- moved G*** 0.19 mm to (129.9, 94.5)
Connections:
- J204 pad 5: /ESP32/GPIO10 -> +3V3
- J204 pad 6: /ESP32/GPIO9 -> +5V
- J204 pad 7: /ESP32/GPIO18 -> /ESP32/GPIO10
- J204 pad 8: /ESP32/GPIO8 -> /ESP32/GPIO9
- J401 pad 10: /ESP32/COMM -> /ESP32/GPIO17
- J401 pad 3: /ESP32/GPIO10 -> /Raspberry Pi/RASP_SDA
- J401 pad 5: /ESP32/GPIO9 -> /Raspberry Pi/RASP_SCL
- R211 pad 2: /ESP32/GPIO18 -> /ESP32/GPIO10
- R212 pad 1: /ESP32/GPIO8 -> /ESP32/GPIO9
- U201 pad 10: /ESP32/COMM -> /ESP32/GPIO17
- U201 pad 12: /ESP32/GPIO8 -> /ESP32/COMM
Routing:
- net /Raspberry Pi/RASP_SCL: track 0.00 -> 56.3 mm, vias 0 -> 1
- net /Raspberry Pi/RASP_SDA: track 0.00 -> 54.4 mm, vias 0 -> 1
- net /ESP32/GPIO17: track 0.00 -> 54.4 mm, vias 0 -> 1
- net /ESP32/COMM: track 73.2 -> 23.9 mm
- net /ESP32/GPIO10: track 84.5 -> 47.3 mm
- net /ESP32/GPIO9: track 75.3 -> 44.0 mm
- net /ESP32/GPIO8: track 26.8 -> 0.00 mm, vias 2 -> 0
- net /ESP32/GPIO18: track 77.0 -> 51.2 mm, vias 2 -> 1
- net /5V_RASP: track 46.0 -> 38.9 mm
- net +5V: track 34.3 -> 36.9 mm
- net +3V3: track 138.6 -> 140.3 mm, vias 4 -> 3
- net /ESP32/CHIP_PU: track 49.2 -> 47.6 mm
- net Net-(JP206-A): track 4.23 -> 5.75 mm
- net Net-(JP207-A): track 4.88 -> 6.38 mm
- net /ESP32/GPIO0: track 13.9 -> 13.3 mm
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- added copper zone on B.Cu, net /5V_RASP
Other:
- board text added: "RASP I2C"

Commit message: Feat: I2C and UART to same pins in ESP32, since any GPIO can be RxD and TxD
Parts:
- added JP103: SolderJumper_2_Open, Jumper:SolderJumper-2_P1.3mm_Bridged_RoundedPad1.0x1.5mm, F.Cu at (169.8, 91.4)
- added JP104: SolderJumper_2_Open, Jumper:SolderJumper-2_P1.3mm_Bridged_RoundedPad1.0x1.5mm, F.Cu at (172.3, 91.4)
- added R401: 4k7, Resistor_SMD:R_0805_2012Metric, F.Cu at (167.2, 87.0)
- added R402: 4k7, Resistor_SMD:R_0805_2012Metric, F.Cu at (165.3, 87.0)
- moved JP101 2.80 mm to (172.3, 87.0)
- moved JP102 2.80 mm to (169.8, 87.0)
- moved R211 1.36 mm to (163.4, 87.0)
- moved R212 1.36 mm to (161.5, 87.0)
Connections:
- J401 pad 10: /ESP32/GPIO17 -> /Raspberry Pi/RASP_RX
- J401 pad 8: /ESP32/GPIO18 -> /Raspberry Pi/RASP_TX
- JP101 pad 2: /ESP32/GPIO9 -> /ESP32/GPIO18
- JP102 pad 2: /ESP32/GPIO10 -> /ESP32/GPIO17
Routing:
- net /Raspberry Pi/RASP_RX: track 0.00 -> 78.3 mm, vias 0 -> 1
- net /Raspberry Pi/RASP_TX: track 0.00 -> 75.5 mm, vias 0 -> 1
- net /ESP32/GPIO17: track 54.4 -> 20.6 mm, vias 1 -> 2
- net /ESP32/GPIO18: track 51.2 -> 23.2 mm, vias 1 -> 2
- net /Raspberry Pi/RASP_SCL: track 56.3 -> 67.8 mm
- net /ESP32/GPIO9: track 44.0 -> 35.3 mm
- net /Raspberry Pi/RASP_SDA: track 54.4 -> 60.9 mm
- net +3V3: track 140.3 -> 145.7 mm
- net /ESP32/GPIO10: track 47.3 -> 43.4 mm
Other:
- board text added: "RASP UART"

Commit message: Feat: final revision
Parts:
- moved C201 3.55 mm to (164.1, 104.7)
- moved G*** 3.45 mm to (162.4, 108.3), turned to 180 degrees
- moved C202 2.21 mm to (164.1, 102.7), turned to 180 degrees
- moved C203 1.24 mm to (161.1, 100.8), turned to 90 degrees
- moved U201 0.38 mm to (150.0, 98.8)
- moved TP201 0.38 mm to (152.0, 86.6)
Connections:
- C211 pad 2: Net-(U202-VDD5) -> +3V3
- C212 pad 2: Net-(U202-VIO) -> +3V3
- JP202 pad 1: /ESP32/U0RXD -> /ESP32/U0TXD
- JP203 pad 1: /ESP32/U0TXD -> /ESP32/U0RXD
- U201 pad 27: unconnected-(U201-GPIO0/BOOT-Pad27) -> /ESP32/GPIO0
- U202 pad 1: Net-(U202-VIO) -> +3V3
- U202 pad 3: Net-(U202-VDD5) -> +3V3
Routing:
- net /ESP32/GPIO0: track 13.3 -> 41.0 mm, vias 1 -> 2
- net +3V3: track 145.7 -> 160.5 mm, vias 3 -> 5
- net Net-(JP202-B): track 9.96 -> 17.3 mm
- net Net-(U202-VDD5): track 4.65 -> 0.00 mm
- net /ESP32/U0TXD: track 23.7 -> 26.3 mm
- net GND: track 6.09 -> 3.56 mm
- net Net-(U202-VIO): track 2.46 -> 0.00 mm
- net /ESP32/U0RXD: track 32.3 -> 31.3 mm
