File: seebum_peripherals/seebum_peripherals.kicad_pcb (KiCad board)
At the start: 2 copper layers, 65 x 56 mm, 48 parts, among them J101 Conn_01x06_Socket, J102 Conn_01x06_Socket, J103 Conn_01x03_Socket, J104 Conn_01x02_Socket, J105 Conn_01x02_Socket, J106 Conn_01x07_Socket, J107 Conn_01x04_Socket, J108 Conn_01x03_Socket, J109 Conn_02x10_Odd_Even, J110 Conn_02x10_Odd_Even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

Commit message: Feat: fix I2C and silkscreen
Parts:
- moved G*** 0.27 mm to (160.6, 101.0)
Connections:
- net /I2C1_SCL renamed /I2C_SCL
- net /I2C1_SDA renamed /I2C_SDA
- J110 pad 5: /I2C0_SDA -> +3V3
- J110 pad 6: /I2C0_SCL -> +5V
Routing:
- net +5V: track 29.6 -> 32.1 mm
- net +3V3: track 195.8 -> 198.4 mm

Commit message: Feat: final revision
Parts:
- moved G*** 5.16 mm to (142.3, 95.6)
Changed lines of the file:
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@@
 			)
 		)
-		(property "Footprint" ""
+		(property "Footprint" "LOGO"
 			(at 0 0 90)
 			(unlocked yes)
@@
 			)
 		)
-		(property "Footprint" ""
+		(property "Footprint" "LOGO"
 			(at 0 0 -90)
 			(unlocked yes)
@@
 			)
 		)
-		(property ki_fp_filters "Connector*:*_2x??_*")
-		(sheetname "Root")
-		(sheetfile "seebum_peripherals.kicad_sch")
 		(attr through_hole)
 		(fp_line
@@
 				(type solid)
 			)
-			(layer "F.SilkS")
+			(layer "B.SilkS")
 		)
 		(fp_line
@@
 				(type solid)
 			)
-			(layer "F.SilkS")
+			(layer "B.SilkS")
 		)
 		(fp_line
@@
 				(type solid)
 			)
-			(layer "F.SilkS")
+			(layer "B.SilkS")
 		)
 		(fp_line
@@
 				(type solid)
 			)
-			(layer "F.SilkS")
+			(layer "B.SilkS")
 		)
 		(fp_line
@@
 				(type solid)
 			)
-			(layer "F.SilkS")
+			(layer "B.SilkS")
 		)
 		(fp_line
@@
 				(type solid)
 			)
-			(layer "F.SilkS")
+			(layer "B.SilkS")
 		)
 		(fp_line
@@
 				(type solid)
 			)
-			(layer "F.SilkS")
+			(layer "B.SilkS")
 		)
 		(fp_line
@@
 				(type solid)
 			)
-			(layer "F.SilkS")
+			(layer "B.SilkS")
 		)
 		(fp_line
@@
 			)
 		)
-		(property "Footprint" ""
+		(property "Footprint" "LOGO"
 			(at 0 0 90)
 			(unlocked yes)
@@
 			)
 		)
-		(property "Footprint" ""
+		(property "Footprint" "LOGO"
 			(at 0 0 90)
 			(unlocked yes)
@@
 			)
 		)
-		(property "Footprint" ""
+		(property "Footprint" "LOGO"
 			(at 0 0 0)
 			(unlocked yes)
@@
 			)
 		)
-		(property "Footprint" ""
+		(property "Footprint" "LOGO"
 			(at 0 0 90)
 			(unlocked yes)
@@
 			)
 		)
-		(property "Footprint" ""
+		(property "Footprint" "LOGO"
 			(at 0 0 90)
 			(unlocked yes)
@@
 			)
 		)
-		(property "Footprint" ""
+		(property "Footprint" "LOGO"
 			(at 0 0 90)
 			(unlocked yes)
@@
 			)
 		)
-		(property "Footprint" ""
+		(property "Footprint" "LOGO"
 			(at 0 0 90)
 			(unlocked yes)
@@
 			)
 		)
-		(property "Footprint" ""
+		(property "Footprint" "LOGO"
 			(at 0 0 90)
 			(unlocked yes)
@@
 			)
 		)
-		(property "Footprint" ""
+		(property "Footprint" "LOGO"
 			(at 0 0 90)
 			(unlocked yes)
@@
 			)
 		)
-		(property "Footprint" ""
+		(property "Footprint" "LOGO"
 			(at 0 0 90)
 			(unlocked yes)
@@
 			)
 		)
-		(property ki_fp_filters "Connector*:*_2x??_*")
-		(sheetname "Root")
-		(sheetfile "seebum_peripherals.kicad_sch")
 		(attr through_hole)
 		(fp_line
@@
 				(type solid)
 			)
-			(layer "F.SilkS")
+			(layer "B.SilkS")
 		)
 		(fp_line
@@
 				(type solid)
 			)
-			(layer "F.SilkS")
+			(layer "B.SilkS")
 		)
 		(fp_line
@@
 				(type solid)
 			)
-			(layer "F.SilkS")
+			(layer "B.SilkS")
 		)
 		(fp_line
@@
 				(type solid)
 			)
-			(layer "F.SilkS")
+			(layer "B.SilkS")
 		)
 		(fp_line
@@
 				(type solid)
 			)
-			(layer "F.SilkS")
+			(layer "B.SilkS")
 		)
 		(fp_line
@@
 				(type solid)
 			)
-			(layer "F.SilkS")
+			(layer "B.SilkS")
 		)
 		(fp_line
@@
 				(type solid)
 			)
-			(layer "F.SilkS")
+			(layer "B.SilkS")
 		)
 		(fp_line
@@
 				(type solid)
 			)
-			(layer "F.SilkS")
+			(layer "B.SilkS")
 		)
 		(fp_line
@@
 			)
 		)
-		(property "Footprint" ""
+		(property "Footprint" "LOGO"
 			(at 0 0 180)
 			(unlocked yes)
@@
 	(footprint "LOGO"
 		(layer "B.Cu")
-		(at 142.3 90.45)
+		(at 142.29 95.61)
 		(property "Reference" "G***"
 			(at 0 0 0)
@@
 			)
 		)
-		(property "Footprint" ""
+		(property "Footprint" "LOGO"
 			(at 0 0 180)
 			(unlocked yes)
@@
 			)
 		)
-		(property "Footprint" ""
+		(property "Footprint" "LOGO"
 			(at 0 0 180)
 			(unlocked yes)
@@
 				(pts
 					(xy 168.315 75.710188) (xy 168.220233 75.744748) (xy 168.220233 75.953332) (xy 168.315 75.987892)
-					(xy 168.315 76.095725) (xy 167.834452 75.911322) (xy 167.834452 75.851238) (xy 167.925554 75.851238)
-					(xy 167.949502 75.858388) (xy 167.957062 75.860764) (xy 167.980775 75.86843) (xy 167.991133 75.871877)
-					(xy 168.014488 75.879933) (xy 168.017878 75.881158) (xy 168.13658 75.9239) (xy 168.13658 75.774546)
-					(xy 168.017878 75.817411) (xy 167.99956 75.824005) (xy 167.976309 75.831569) (xy 167.975502 75.831821)
-					(xy 167.951718 75.839125) (xy 167.949246 75.839881) (xy 167.925554 75.847208) (xy 167.925554 75.851238)
-					(xy 167.834452 75.851238) (xy 167.834452 75.782362) (xy 168.315 75.597348)
+					(xy 168.315 76.095725) (xy 167.834452 75.911322) (xy 167.834452 75.847208) (xy 167.925554 75.847208)
+					(xy 167.925554 75.851238) (xy 167.949502 75.858388) (xy 167.957062 75.860764) (xy 167.980775 75.86843)
+					(xy 167.991133 75.871877) (xy 168.014488 75.879933) (xy 168.017878 75.881158) (xy 168.13658 75.9239)
+					(xy 168.13658 75.774546) (xy 168.017878 75.817411) (xy 167.99956 75.824005) (xy 167.976309 75.831569)
+					(xy 167.975502 75.831821) (xy 167.951718 75.839125) (xy 167.949246 75.839881) (xy 167.925554 75.847208)
+					(xy 167.834452 75.847208) (xy 167.834452 75.782362) (xy 168.315 75.597348)
 				)
 			)
@@
 					(xy 168.268078 75.18357) (xy 168.28221 75.204134) (xy 168.28911 75.216939) (xy 168.299198 75.241036)
 					(xy 168.306808 75.267272) (xy 168.311359 75.291462) (xy 168.314089 75.317224) (xy 168.315 75.344556)
-					(xy 168.315 75.540561) (xy 167.834452 75.540561) (xy 167.834452 75.435659) (xy 167.920425 75.435659)
-					(xy 168.229026 75.435659) (xy 168.229026 75.345167) (xy 168.227514 75.320598) (xy 168.222014 75.295305)
-					(xy 168.219867 75.289113) (xy 168.20851 75.266826) (xy 168.192756 75.248569) (xy 168.172545 75.23422)
-					(xy 168.149493 75.224427) (xy 168.147815 75.2239) (xy 168.122564 75.21814) (xy 168.096186 75.21568)
-					(xy 168.085289 75.215474) (xy 168.064651 75.215474) (xy 168.038976 75.216659) (xy 168.013992 75.220617)
-					(xy 168.001758 75.2239) (xy 167.978442 75.233457) (xy 167.957948 75.247554) (xy 167.956817 75.248569)
-					(xy 167.94013 75.268101) (xy 167.929584 75.289113) (xy 167.92301 75.313533) (xy 167.920506 75.339279)
-					(xy 167.920425 75.345167) (xy 167.920425 75.435659) (xy 167.834452 75.435659) (xy 167.834452 75.344556)
+					(xy 168.315 75.540561) (xy 167.834452 75.540561) (xy 167.834452 75.345167) (xy 167.920425 75.345167)
+					(xy 167.920425 75.435659) (xy 168.229026 75.435659) (xy 168.229026 75.345167) (xy 168.227514 75.320598)
+					(xy 168.222014 75.295305) (xy 168.219867 75.289113) (xy 168.20851 75.266826) (xy 168.192756 75.248569)
+					(xy 168.172545 75.23422) (xy 168.149493 75.224427) (xy 168.147815 75.2239) (xy 168.122564 75.21814)
+					(xy 168.096186 75.21568) (xy 168.085289 75.215474) (xy 168.064651 75.215474) (xy 168.038976 75.216659)
+					(xy 168.013992 75.220617) (xy 168.001758 75.2239) (xy 167.978442 75.233457) (xy 167.957948 75.247554)
+					(xy 167.956817 75.248569) (xy 167.94013 75.268101) (xy 167.929584 75.289113) (xy 167.92301 75.313533)
+					(xy 167.920506 75.339279) (xy 167.920425 75.345167) (xy 167.834452 75.345167) (xy 167.834452 75.344556)
 					(xy 167.835366 75.317224) (xy 167.83811 75.291462) (xy 167.842682 75.267272) (xy 167.850328 75.241036)
 					(xy 167.860464 75.216939) (xy 167.873082 75.195033) (xy 167.888283 75.175476) (xy 167.906067 75.158268)
